File: stepper_driver.sch (KiCad schematic (older format))
At the start: 83 parts, among them IC1 TMC2160-TA, J1 BARREL_JACK, J2 Screw_Terminal_01x04, J3 CONN_02X07, J4 CONN_01X04, J9 USB_C_Receptacle_USB2.0, Q1 Q_NPN_BEC, Q2 Si4946BEY, Q3 Si4946BEY, Q4 Q_NPN_BEC, Q5 Si4946BEY, Q6 Si4946BEY, SW1 SW_Push, SW2 SW_Push, U1 CH340B, U2 XC6210B332MR, U3 XL1509-5.0, U4 ESP32-WROOM-32D, U6 SN74LV1T34DBV

Commit message: Updated hardware to rev 3
Parts:
- removed C12: 330uF/16V, Capacitor_SMD:CP_Elec_8x10.5, symbol Device:CP
- removed D1: D_Schottky, Diode_SMD:D_SOD-123, symbol Device:D_Schottky
- removed J4: CONN_01X04, Connector_PinHeader_1.27mm:PinHeader_1x04_P1.27mm_Vertical, symbol conn1:CONN_01X04
- removed U3: XL1509-5.0, Package_SO:SOIC-8_3.9x4.9mm_P1.27mm, symbol xl1509:XL1509
- removed U4: ESP32-WROOM-32D, RF_Module:ESP32-WROOM-32, symbol RF_Module:ESP32-WROOM-32
- removed U6: SN74LV1T34DBV, Package_TO_SOT_SMD:SOT-23-5, symbol Logic_LevelTranslator:SN74LV1T34DBV
- added AE1: KH3216-A55, KH3216:KH3216-A55, symbol Device:Antenna_Chip
- added C12, C33: 10uF/50V, Capacitor_SMD:C_0805_2012Metric, symbol Device:C
- added C28: 1.5pF, Capacitor_SMD:C_0603_1608Metric, symbol Device:C
- added C30: 0.1uF, Capacitor_SMD:C_0402_1005Metric, symbol Device:C
- added C31: 220uF/50V, Capacitor_THT:CP_Radial_D10.0mm_P5.00mm, symbol Device:CP
- added C32: 0.47uF/25V, Capacitor_SMD:C_0402_1005Metric, symbol Device:C
- added C34, C36: 0.1uF/50V, Capacitor_SMD:C_0402_1005Metric, symbol Device:C
- added C35, C37: 10uF/25V, Capacitor_SMD:C_0603_1608Metric, symbol Device:C
- added D1: SMBJ40A, Diode_SMD:D_SMB, symbol Device:D_Zener
- added D5, D6: 60V/1A, Diode_SMD:D_SOD-323F, symbol Device:D_Schottky
- added J5: Conn_Coaxial, Connector_Coaxial:U.FL_Hirose_U.FL-R-SMT-1_Vertical, symbol Connector:Conn_Coaxial
- added JP1: SolderJumper_2_Open, Resistor_SMD:R_0402_1005Metric, symbol Jumper:SolderJumper_2_Open
- added L1: 5.1nH, Inductor_SMD:L_0603_1608Metric, symbol pspice:INDUCTOR
- added L3: 10uH, Inductor_SMD:L_1210_3225Metric, symbol pspice:INDUCTOR
- added R24: 0R, Resistor_SMD:R_0402_1005Metric, symbol Device:R
- added R26: 10kR, Resistor_SMD:R_0402_1005Metric, symbol Device:R
- added R27: 330kR, Resistor_SMD:R_0402_1005Metric, symbol Device:R
- added R28: 24kR, Resistor_SMD:R_0402_1005Metric, symbol Device:R
- added R29, R30, R31, R32: 1R, Resistor_SMD:R_0402_1005Metric, symbol Device:R
- added R33: 120kR, Resistor_SMD:R_0402_1005Metric, symbol Device:R
- added R34: 22kR, Resistor_SMD:R_0402_1005Metric, symbol Device:R
- added U3, U5: TP6841S6-A, Package_TO_SOT_SMD:SOT-23-6, symbol Regulator_Switching:LM2734Y
- added U4: ESP32-PICO-D4, Package_DFN_QFN:QFN-48-1EP_7x7mm_P0.5mm_EP5.3x5.3mm, symbol RF_Module:ESP32-PICO-D4
- C11: value 1uF/50V -> 0.1uF; footprint Capacitor_SMD:C_0603_1608Metric -> Capacitor_SMD:C_0402_1005Metric; LCSC C15849 -> C1525
- C15, C18: LCSC C96446 -> C386081
- C16: value 0.47uF/25V -> 0.1uF; LCSC C437527 -> C1525
- C3: value 470uF/50V -> 220uF/50V; LCSC C106526 -> C88723
- D2, D4: value D_Schottky -> 60V/1A; footprint Diode_SMD:D_SOD-123 -> Diode_SMD:D_SOD-323F; LCSC C8598 -> C364278
- L2: value 68uH -> 10uH; footprint Inductor_SMD:L_Taiyo-Yuden_NR-60xx -> Inductor_SMD:L_1210_3225Metric; LCSC C83460 -> C86069
Connections:
- net +3V3: now also J3.13 (P13), C30.1, R26.2, U4.1 (VDDA), U4.19 (VDD3P3_RTC), U4.3 (VDDA3P3), U4.37 (VDD3P3_CPU), U4.4 (VDDA3P3), U4.43 (VDDA), U4.46 (VDDA); no longer J3.2 (P2)
- net +5V: now also C37.1, L3.2, R33.1; no longer D4.1 (K)
- net BMA1: now also C5.1, D4.1 (K), R29.2; no longer C16.1, C26.1, J2.2 (Pin_2), Q6.1 (S1), Q6.5 (D2), Q6.6 (D2)
- net BMA2: now also D2.1 (K), R30.2; no longer C27.1, J2.1 (Pin_1), Q5.1 (S1), Q5.5 (D2), Q5.6 (D2)
- net BMB1: now also C32.1, D6.1 (K), R31.2; no longer C24.1, C5.1, J2.4 (Pin_4), Q2.1 (S1), Q2.5 (D2), Q2.6 (D2)
- net BMB2: now also D5.1 (K), R32.2; no longer C25.1, J2.3 (Pin_3), Q3.1 (S1), Q3.5 (D2), Q3.6 (D2)
- net CA1: now also C5.2; no longer C16.2
- net CB1: now also C32.2; no longer C5.2
- net EN: now also U4.9 (EN)
- net GND: now also D4.2 (A), J3.2 (P2), C12.2, C28.2, C30.2, C31.2, C33.2, C34.1, C35.2, C36.1, C37.2, D1.2 (A), D5.2 (A), D6.2 (A), J5.2 (Ext), R28.2, R34.2, U3.2 (GND), U4.49 (GND), U5.2 (GND); no longer C11.2, J3.13 (P13)
- net I34: now also J3.6 (P6), U4.10 (IO34); no longer J3.4 (P4)
- net I35: now also J3.8 (P8), U4.11 (IO35); no longer J3.5 (P5)
- net I39: now also J3.4 (P4), U4.8 (SENSOR_VN); no longer J3.3 (P3)
- net IO0: now also U4.23 (IO0)
- net IO12: now also U4.18 (IO12); no longer J3.12 (P12)
- net IO14: now also J3.9 (P9), U4.17 (IO14); no longer J3.11 (P11)
- net IO27: now also J3.11 (P11), U4.16 (IO27); no longer J3.10 (P10)
- net IO32: now also J3.10 (P10), U4.12 (IO32); no longer J3.6 (P6)
- net IO33: now also J3.12 (P12), U4.13 (IO33); no longer J3.7 (P7)
- net LED_DATA: now also D3.4 (DIN), U4.42 (IO21)
- net PAIR_SW: now also U4.39 (IO22)
- net TMC_CLK: now also U4.35 (IO18)
- net TMC_CS: now also U4.34 (IO5)
- net TMC_DCEN: now also U4.29 (SD3/IO10)
- net TMC_DCO: now also U4.28 (SD2/IO9)
- net TMC_DIAG0: now also U4.24 (IO4)
- net TMC_DIAG1: now also U4.22 (IO2)
- net TMC_DIR: now also J3.5 (P5), U4.15 (IO26); no longer J3.9 (P9)
- net TMC_MISO: now also U4.38 (IO19)
- net TMC_MOSI: now also U4.36 (IO23)
- net TMC_STEP: now also J3.3 (P3), U4.14 (IO25); no longer J3.8 (P8)
- net TMC_~EN: now also R26.1, U4.21 (IO15)
- net USB_TX: now also U4.40 (U0RXD/IO3)
- net VS: now also C12.1, C31.1, C33.1, C34.2, C36.2, D1.1 (K), U3.4 (EN), U3.5 (VIN), U5.4 (EN), U5.5 (VIN); no longer C1.1, C11.1, IC1.4 (VSA)
- net VS_SENSE: now also U4.5 (SENSOR_VP)
- net at R25.2: now also U4.41 (U0TXD/IO1)
- net at L2.1: now also C11.2, U3.6 (SW); no longer D2.1 (K)
- net +12V: now reaches L2.2
- net +12V: now also C1.1, IC1.4 (VSA), C35.1, R27.1; no longer D4.2 (A)
- new net: J5.1 (In), JP1.2 (B)
- new net: C11.1, U3.1 (BOOST)
- new net: R27.2, R28.1, U3.3 (FB)
- new net: C16.1, U5.1 (BOOST)
- new net: R33.2, R34.1, U5.3 (FB)
- new net: C16.2, L3.1, U5.6 (SW)
- new net ANT: C28.1, JP1.1 (A), L1.1, R24.1
- new net ANT_OUT: AE1.1 (FEED), L1.2
- new net AO1: C26.1, J2.2 (Pin_2), Q6.1 (S1), Q6.5 (D2), Q6.6 (D2), R29.1
- new net AO2: C27.1, J2.1 (Pin_1), Q5.1 (S1), Q5.5 (D2), Q5.6 (D2), R30.1
- new net BO1: C24.1, J2.4 (Pin_4), Q2.1 (S1), Q2.5 (D2), Q2.6 (D2), R31.1
- new net BO2: C25.1, J2.3 (Pin_3), Q3.1 (S1), Q3.5 (D2), Q3.6 (D2), R32.1
- new net IO13: J3.7 (P7), U4.20 (IO13)
- new net LNA: R24.2, U4.2 (LNA_IN)
- no-connect marks 6 -> 7
Other:
- note added: "Antenna"
- note added: "JLC2313 Substrate Microstrip:\n5.78 mil trace (11.55 mil for JLC7628)\nMin 17 mil space (35 mil for JLC7628)\nZ0 = 50R"
- note added: "Requirements:\nBLE: 2.400 – 2.4835 GHz\nWiFi: 2.401 - 2.495 GHz"
- note removed: "Gate Drive Tuning"
- moved on the sheet: C17, C22, C23, C24, C25, C26, C27, C3, C7, C8, C9, H1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

Commit message: Rev3 PCB tweaks
Parts:
- added C29, C38: 2.2nF, Capacitor_SMD:C_0402_1005Metric, symbol Device:C
- added C39, C40: 0.1uF, Capacitor_SMD:C_0402_1005Metric, symbol Device:C
- added H10: MountingHole, Symbol:OSHW-Logo_5.7x6mm_SilkScreen, symbol Mechanical:MountingHole
- added H9: MountingHole, Symbol:Symbol_Barrel_Polarity, symbol Mechanical:MountingHole
- added R35: 1R, Resistor_SMD:R_0402_1005Metric, symbol Device:R
- added R36, R37: 100kR, Resistor_SMD:R_0402_1005Metric, symbol Device:R
- C11, C16: value 0.1uF -> 0.22uF; LCSC C1525 -> C16772
- C21: value 0.1uF/50V -> 0.22uF/50V; footprint Capacitor_SMD:C_0603_1608Metric -> Capacitor_SMD:C_0805_2012Metric; LCSC C14663 -> C5378
- L2, L3: value 10uH -> 22uH; LCSC C86069 -> C223225
- R22: value 470R -> 150R; LCSC C25117 -> C25082
Connections:
- net +12V: now also C15.2, IC1.3 (12VOUT)
- net GND: now also C39.2, C40.2
- net SRAH: now also C29.1
- net SRAL: now also C29.2
- net SRBH: now also C38.1
- net SRBL: now also C38.2
- net VS: now also R35.2, R36.2, R37.2; no longer C14.2, C21.1, IC1.33 (VS), U3.4 (EN), U5.4 (EN)
- net at Q2.3 (S2), Q3.3 (S2), R1.1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: now also C40.1
- net at Q5.3 (S2), Q6.3 (S2), R19.1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: now also C39.1
- new net: C14.2, C21.1, IC1.33 (VS), R35.1
- new net: R37.1, U5.4 (EN)
- new net: R36.1, U3.4 (EN)
Other:
- note added: "OSHW"
- note added: "Polarity"
- note added: "Symbols"
- moved on the sheet: AE1, C12, C13, C21, C28, C32, C33, C34, C36, C5, D3, D4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

Commit message: Cosmetics update
Parts:
- JP1: value SolderJumper_2_Open -> Open
Connections:
- net ANT: no longer names the net of C28.1, JP1.1 (A), L1.1, R24.1
- net CC1: no longer names the net of J9.A5 (CC1), R3.1
- net CC2: no longer names the net of J9.B5 (CC2), R13.1
- net Dm: no longer names the net of J9.A7 (D-), J9.B7 (D-), U1.6 (UD-)
- net Dp: no longer names the net of J9.A6 (D+), J9.B6 (D+), U1.5 (UD+)
- no-connect marks 7 -> 8
Other:
- moved on the sheet: C13, C28, C30, C4, C9, D1, J5, JP1, R13, R21, R22, R23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

Commit message: Finalised rev3 files
Parts:
- removed AE1: KH3216-A55, KH3216:KH3216-A55, symbol Device:Antenna_Chip
- removed H1: MountingHole, MountingHole:MountingHole_3.5mm, symbol Mechanical:MountingHole
- removed L1: 5.1nH, Inductor_SMD:L_0603_1608Metric, symbol pspice:INDUCTOR
- added AE1: IFA Antenna, Antennas:TI_DN007_2.4GHz, symbol Device:Antenna_Dipole
- added R38: 0R, Resistor_SMD:R_0603_1608Metric, symbol Device:R
- C12, C33: footprint Capacitor_SMD:C_0805_2012Metric -> Capacitor_SMD:C_1206_3216Metric; LCSC C440198 -> C13585
- C28: value 1.5pF -> DNP; LCSC C519100 -> (none)
- D1: value SMBJ40A -> SMBJ36A; LCSC C309963 -> C294880
- J9: footprint Connector_USB:USB_C_Receptacle_HRO_TYPE-C-31-M-12 -> Connector_USB:USB_C_Receptacle_XKB_U262-16XN-4BVC11; LCSC C165948 -> C319148
- Q2, Q3, Q5, Q6: value Si4946BEY -> NCE6005AS; LCSC C83862 -> C126151
- R10, R11, R12, R14, R15, R5, R7, R8: value 10R -> 4.7R; LCSC C25077 -> C25121
- R25: value 470R -> 150R; LCSC C25117 -> C25082
- R29, R30, R31, R32, R35: LCSC C25077 -> C25086
- U4: footprint Package_DFN_QFN:QFN-48-1EP_7x7mm_P0.5mm_EP5.3x5.3mm -> ESP32-PICO-D4:ESP32-PICO-D4; LCSC (none) -> C193707
Connections:
- net ANT_OUT: now also AE1.2, R38.1
- net GND: now also AE1.1
- net at C28.1, JP1.1 (A), R24.1: now also R38.2
Other:
- note added: "BLE: 2.400 – 2.4835 GHz\nWiFi: 2.401 - 2.495 GHz"
- note added: "Grounded Coplanar Wave Guide (JLC7628 Substrate):\nCalculator: https://spok.ca/index.php/resources/tools/99-cpwcalc\nH = 0.18, W=0.295, T=0.035, S=0.2, Er=4.6, Z0 = 50.05R\n\nVerified with TNT MMTL Sim: See doc/tline_analysis/1mm_gcpw"
- note added: "HIGH ON BOOT (MTDO)"
- note added: "HIGH ON BOOT (STRAPPING)"
- note added: "LOW ON BOOT (STRAPPING)"
- note removed: "JLC2313 Substrate Microstrip:\n5.78 mil trace (11.55 mil for JLC7628)\nMin 17 mil space (35 mil for JLC7628)\nZ0 = 50R"
- note removed: "Requirements:\nBLE: 2.400 – 2.4835 GHz\nWiFi: 2.401 - 2.495 GHz"
- moved on the sheet: C22, C23, C30, C9, R21, R22, R23, R25, SW2, U4
